Commit message: Modified prefix on robotic arm

File: kinova_robot_arm_description/urdf/gen3_lite_gen3_lite_2f.xacro (robot description, xacro)
@@ -7,5 +7,5 @@
   <xacro:property name="gripper" value="gen3_lite_2f" />
   <xacro:property name="parent" default="world" />
-  <xacro:property name="prefix" default="kinova" />
+  <xacro:property name="prefix" default="kinova_" />
   <!-- Define the load_robot macros -->
   <xacro:macro name="load_robot" params="
